File: Modulo_SIMA7670SA.kicad_pcb (KiCad board)
At the start: 2 copper layers, 90.3 x 85 mm, 57 parts, among them J1 TBP01R1-508-02BE, J2 DB9 Hembra Impreso 90°, J3 U.FL IPEX1 MALE, J4 SMA-J-P-X-RA-TH1, J5 Jack DC 2.1mm PCB recto, Q1 BSS138, Q2 FDN340P, Q3 FDN340P, Q4 BSS138, U1 MAX232, U2 24LC512, U3 BKP-A7670SA (Módulo SIMCOM), U5 Black_Pill_STM32F411CEUx, U6 LM2596S_Modulo_Regulable, U7 LM7805_TO220

Commit message: Reforzamos un poco más la conexión GND del step-down
Routing:
- net GND: track 316.4 -> 332.7 mm
Changed lines of the file:
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@@
+	)
+	(segment
+		(start 143.36 78.16)
+		(end 143.26 78.26)
+		(width 2.5)
+		(layer "B.Cu")
+		(net "GND")
 	)
 	(segment
@@
 	)
 	(segment
+		(start 154.86 82.66)
+		(end 150.46 78.26)
+		(width 2.5)
+		(layer "B.Cu")
+		(net "GND")
+	)
+	(segment
 		(start 190.66 137.66)
 		(end 190.66 140.68)
@@
 		(end 135.66 89.66)
 		(width 2)
+		(layer "B.Cu")
+		(net "GND")
+	)
+	(segment
+		(start 143.36 75.36)
+		(end 143.36 78.16)
+		(width 2.5)
 		(layer "B.Cu")
 		(net "GND")
@@
 		(layer "B.Cu")
 		(net "GND")
+	)
+	(segment
+		(start 150.46 78.26)
+		(end 143.26 78.26)
+		(width 2.5)
+		(layer "B.Cu")
+		(net "GND")
