File: Modulo_SIMA7670SA.kicad_pcb (KiCad board)
At the start: 2 copper layers, 90.3 x 85 mm, 57 parts, among them J1 TBP01R1-508-02BE, J2 DB9 Hembra Impreso 90°, J3 U.FL IPEX1 MALE, J4 SMA-J-P-X-RA-TH1, J5 Jack DC 2.1mm PCB recto, Q1 BSS138, Q2 FDN340P, Q3 FDN340P, Q4 BSS138, U1 MAX232, U2 24LC512, U3 BKP-A7670SA (Módulo SIMCOM), U5 Black_Pill_STM32F411CEUx, U6 LM2596S_Modulo_Regulable, U7 LM7805_TO220

Commit message: Se hicieron los arreglos para hacer funcionar el visor 3D de kicad 10.0.3. Comenzamos a tirar las primeras líneas del Gabinete basándonos en el modelo 3D.
Parts:
- moved J1 4.97 mm to (143.6, 65.2), turned to 180 degrees
Connections:
- J1 pad 1: GND -> +12V
- J1 pad 2: +12V -> GND

Commit message: Rediseño HW: separación de dominios de alimentación y actualización de footprints - Riel 12V/5V del modem independiente (12V_StepDown→FDN340P→5V_MODEM): brownout resuelto y validado en PCB - Switches BC327/BC547 → topología FDN340P; MV5439A sustituido por WP59EGW/CA - Footprints en Damian_PCB: BKP-A7670SA, MF-NSMF005/60X, SM15-02HTG; corregido tamaño de pads del barrel jack - RS232: modificaciones incorporadas al esquema (pendiente pasar a PCB)
Changed lines of the file:
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@@
 		(grid_origin 114.86 145.66)
 		(pcbplotparams
-			(layerselection 0x00000000_00000000_55555555_5755f57f)
+			(layerselection 0x00000000_00000000_5555555d_d7557577)
 			(plot_on_all_layers_selection 0x00000000_00000000_00000000_02000000)
 			(disableapertmacros no)
@@
 		(sheetname "/")
 		(sheetfile "Modulo_SIMA7670SA.kicad_sch")
-		(units
-			(unit
-				(name "A")
-				(pins "MP" "1" "2")
-			)
-		)
 		(attr through_hole)
 		(duplicate_pad_numbers_are_jumpers no)
@@
 		(pad "1" thru_hole rect
 			(at 0 0 180)
-			(size 2.6 2.6)
-			(drill 1.6)
+			(size 4 3)
+			(drill oval 3.5 1.2)
 			(layers "*.Cu" "*.Mask")
 			(remove_unused_layers no)
@@
 			(pintype "passive")
 		)
-		(pad "2" thru_hole circle
+		(pad "2" thru_hole rect
 			(at 0 6 180)
-			(size 2.6 2.6)
-			(drill 1.6)
+			(size 4 2)
+			(drill oval 3 1.2)
 			(layers "*.Cu" "*.Mask")
 			(remove_unused_layers no)
@@
 			(pintype "passive")
 		)
-		(pad "3" thru_hole circle
+		(pad "3" thru_hole rect
 			(at 4.7 3 180)
-			(size 2.6 2.6)
-			(drill 1.6)
+			(size 3 4.5)
+			(drill oval 1.2 3)
 			(layers "*.Cu" "*.Mask")
 			(remove_unused_layers no)
